File: PWR/PWR.kicad_sch (KiCad schematic)
At the start: 17 parts, among them J1 +12v, SW1 SPDT

Commit message: feat: Replaced the pin header by a terminal block. Changed the LEDs labels.
Parts:
- DS1: value GREEN -> ADAPTER
- DS2: value ORANGE -> BATTERY
- DS3: value RED -> STANDBY
- J2: footprint XS:Connector-Breakaway-Header-2.54x0.66mm-2 -> XS:Connector-Wurth-Terminal-Block-2P-3.5mm-691214110002
Changed lines of the file:
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@@
       (effects (font (size 1.27 1.27)))
     )
-    (property "Value" "RED" (at 123.5075 120.65 0)
+    (property "Value" "STANDBY" (at 123.5075 120.65 0)
       (effects (font (size 1.27 1.27)))
     )
@@
       (effects (font (size 1.27 1.27)) (justify left) hide)
     )
-    (property "Footprint" "XS:Connector-Breakaway-Header-2.54x0.66mm-2" (at 219.71 106.68 0)
+    (property "Footprint" "XS:Connector-Wurth-Terminal-Block-2P-3.5mm-691214110002" (at 219.71 106.68 0)
       (effects (font (size 1.27 1.27)) hide)
     )
@@
       (effects (font (size 1.27 1.27)))
     )
-    (property "Value" "ORANGE" (at 123.5075 88.9 0)
+    (property "Value" "BATTERY" (at 123.5075 88.9 0)
       (effects (font (size 1.27 1.27)))
     )
@@
       (effects (font (size 1.27 1.27)))
     )
-    (property "Value" "GREEN" (at 123.5075 76.2 0)
-      (effects (font (size 1.27 1.27)))
-    )
+    (property "Value" "ADAPTER" (at 123.5075 76.2 0)
+      (effects (font (size 1.27 1.27)))
+    )

Commit message: fix: Changed standby LED to 1K
Parts:
- R3: value 100K -> 1K
Changed lines of the file:
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@@
       (effects (font (size 1.27 1.27)))
     )
-    (property "Value" "100K" (at 132.08 121.92 90)
+    (property "Value" "1K" (at 132.08 121.92 90)
       (effects (font (size 1.27 1.27)))
     )
